File: platine/_saved_swr_meter.sch (KiCad schematic (older format))
At the start: 16 parts, among them U1 CP0x0xx5425xNTR_Directional_C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, U2 LTC5530, U3 LM1117_SOT223, U4 STM32F030C8Tx

Commit message: worked on schematic and started pcb
Parts:
- U1: footprint (none) -> Toni:CP0603_directional_coupler
Changed lines of the file:
@@
 F 0 "U1" H 3050 2400 60  0000 C CNN
 F 1 "CP0x0xx5425xNTR_Directional_Coupler" H 3250 1900 60  0000 C CNN
-F 2 "" H 2500 2600 60  0001 C CNN
+F 2 "Toni:CP0603_directional_coupler" H 2500 2600 60  0001 C CNN
 F 3 "" H 2500 2600 60  0000 C CNN
 	1    3050 2150
