File: platine/swr_meter.sch (KiCad schematic (older format))
At the start: 35 parts, among them P1 Oled, P2 Vin, U1 CP0x0xx5425xNTR_Directional_C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, U2 LTC5530, U3 LM1117_SOT223, U4 STM32F030C8Tx, U5 STM32_mmvisual_JTAG, U6 74HC595, U7 74HC595, Y1 8 MHz

Commit message: perhaps not correctly saved bevore the last commit.
Parts:
- added R6, R7: 3,3k, Resistors_SMD:R_0603, symbol R
Connections:
- net +3V3: now also R6.1, R7.1
- net oled_scl: now also R7.2
- net oled_sda: now also R6.2
Changed lines of the file:
@@
 oled_scl
 Wire Wire Line
-	1000 6400 1550 6400
+	850  6400 1550 6400
 Wire Wire Line
-	1550 6500 1000 6500
+	650  6500 1550 6500
 NoConn ~ 1550 4800
 NoConn ~ 1550 4700
@@
 Wire Wire Line
 	8850 1250 9000 1250
+$Comp
+L R R7
+U 1 1 57117F4D
+P 850 6250
+F 0 "R7" V 930 6250 50  0000 C CNN
+F 1 "3,3k" V 850 6250 50  0000 C CNN
+F 2 "Resistors_SMD:R_0603" V 780 6250 50  0001 C CNN
+F 3 "" H 850 6250 50  0000 C CNN
+	1    850  6250
+	1    0    0    -1
+$EndComp
+$Comp
+L R R6
+U 1 1 5711815D
+P 650 6350
+F 0 "R6" V 730 6350 50  0000 C CNN
+F 1 "3,3k" V 650 6350 50  0000 C CNN
+F 2 "Resistors_SMD:R_0603" V 580 6350 50  0001 C CNN
+F 3 "" H 650 6350 50  0000 C CNN
+	1    650  6350
+	1    0    0    -1
+$EndComp
+$Comp
+L +3.3V #PWR046
+U 1 1 571184FE
+P 650 6200
+F 0 "#PWR046" H 650 6050 50  0001 C CNN
+F 1 "+3.3V" H 650 6340 50  0000 C CNN
+F 2 "" H 650 6200 50  0000 C CNN
+F 3 "" H 650 6200 50  0000 C CNN
+	1    650  6200
+	1    0    0    -1
+$EndComp
+$Comp
+L +3.3V #PWR047
+U 1 1 5711877E
+P 850 6100
+F 0 "#PWR047" H 850 5950 50  0001 C CNN
+F 1 "+3.3V" H 850 6240 50  0000 C CNN
+F 2 "" H 850 6100 50  0000 C CNN
+F 3 "" H 850 6100 50  0000 C CNN
+	1    850  6100
+	1    0    0    -1
+$EndComp
 $EndSCHEMATC
